File: apps/web/public/hardware/oapogee.kicad_sch (KiCad schematic)
At the start: 56 parts, among them J1 USB-C-16P, J2 S2B-PH-K-S, J3 ANT-902-928, SW1 ARM-SWITCH, U1 MCP73831, U2 TODO-BUCK-BOOST, U3 RP2350A, U4 W25Q128JVSIQ, U5 BMP390, U6 ICM-42688-P, U7 ADXL375, U8 SX1262, U9 MAX-M10S

Commit message: The board could be flashed once and then never again
A page verification pass across the whole site found a hardware defect, which is
not where I expected one to come from.

RUN, SWCLK and SWDIO were all NOT_CONNECTED in the generated netlist, and
QSPI_CS went only to the flash. There is no dedicated bootloader pin on this
microcontroller: holding the flash chip select low as the chip leaves reset is
what selects USB boot. So a fabricated board could have been programmed exactly
once, while its flash was still blank and the bootrom fell through to USB, and
after that there would have been no way into the bootloader, no way to reset it,
and no way to attach a debugger. For a payload meant to be reflashed between
flights that is fatal, and I published Gerbers for it.

It was invisible in the schematic because the pins were simply absent, and
invisible to every check because nothing asserts that a microcontroller can be
programmed. Three pages meanwhile told the reader to "hold the boot button",
which is how it was caught: an instruction referring to a part that does not
exist.

The board now has SW2 on the flash chip select, SW3 on RUN, R9 pulling RUN up,
and three SWD pads. Press and hold boot, tap reset, release boot. It still
routes: 31 components, 108 traces, 152 vias, no missing traces, no unconnected
ports, no placement errors, and the fabrication package regenerated. The build
guide, the firmware page and the troubleshooting entry now describe what those
buttons actually do, including that a blank board enumerates on its own so the
first flash works even with an unsoldered button, which is exactly the sort of
thing that hides a missing part until the second flash.

The schematic page carried a red callout saying the pin numbers were structural
placeholders and "do not send anything here to a fabricator", twenty lines above
a Files tab offering the Gerbers and a heading saying the board can be ordered.
Both cannot be true. The pin numbers stopped being placehold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
Parts:
- removed GND (x13): GND, symbol Custom:rail_down
- removed V3V3 (x11): V3V3, symbol Custom:rail_up
- removed VBAT (x4): VBAT, symbol Custom:rail_up
- added GND (x5): GND, symbol Custom:rail_down
- added J4: SWD-PADS, symbol Device:U_SWD-PADS
- added R9: 10kΩ, symbol Device:boxresistor_right
- added SW2: BOOT-BUTTON, symbol Device:U_BOOT-BUTTON
- added SW3: RESET-BUTTON, symbol Device:U_RESET-BUTTON
Connections:
- net GND: now also C2.2, C3.2, R1.2, R2.2, R8.2, U2.2 (GND), U4.4 (GND), U6.2 (GND), U7.2 (GND), U8.2 (GND), SW2.3 (B1), SW2.4 (B2), SW3.3 (B1), SW3.4 (B2)
- net VBAT: now reaches J2.1 (VBAT), R7.1
- net VBAT: now also C1.1, U1.3 (VBAT), U2.1 (VIN), U2.3 (EN)
- net V3V3: now reaches R4.2, R5.2
- net V3V3: now also C2.1, C3.1, D1.2 (VDD), R6.2, U2.4 (VOUT), U3.1 (VDD), U4.8 (VCC), U5.1 (VDD), U6.1 (VDD), U7.1 (VDD), U8.1 (VDD), U9.1 (VCC), R9.1
- net at SW1.2 (B): now also J4.3 (GND)
- net U3_QSPI_CS: now reaches U3.60 (QSPI_CS), U4.1 (CS)
- net U3_QSPI_CS: now also SW2.1 (A1), SW2.2 (A2)
- net U3_RUN: now reaches U3.26 (RUN)
- net U3_RUN: now also R9.2, SW3.2 (A2)
- new net U3_SWCLK: J4.1 (SWCLK)
- new net U3_SWDIO: J4.2 (SWDIO)

Commit message: Choose the regulator, and find out the board had outgrown itself
U2 was manufacturerPartNumber="TODO-BUCK-BOOST" on a five pin SOT-23, which is a
placeholder standing in for the part that feeds everything else. It is a
TPS63001 now, and every figure behind that choice comes from TI's datasheet
SLVS520C rather than from memory: 1.8 V to 5.5 V in, which spans a single
lithium cell from full charge to cutoff; fixed 3.3 V out, so there is no
feedback divider and no resistor pair to get wrong; up to 800 mA; 40 uA typical
quiescent at no load; VSON-10, 3 by 3 mm, exposed pad to PGND; one external
2.2 uH inductor, which is now L2.

Quiescent current decided it rather than efficiency at load. This payload sits
armed on a pad and then beeps in a field, both at almost no draw, so standing
loss is what sets how long it keeps beeping.

The schematic carries the datasheet's own pin numbering, the pad tied to PGND,
FB tied to VOUT as fixed-output parts require, and PS/SYNC grounded to enable
power-save, which is the mode that matters for a payload spending hours near
zero load.

Choosing it exposed something else. Adding eleven pads and two parts to a 22 by
60 mm board took the autorouter from seconds to over ten minutes, and then to
not finishing at all: a run was killed after forty-three minutes still working
on the schematic export. That is not a slow build, it is a build that cannot be
relied on to complete. The board is 28 by 78 mm with the placement spread to
match, which routes in under a minute, and the closest copper improved from
0.108 to 0.115 mm and the closest copper to a board edge from 0.72 to 1.34 mm as
a side effect. 32 components, 115 traces, 153 vias, nothing missing, nothing
unconnected, no placement errors, and the fabrication package regenerated. It
still fits the BT-55 sled, with 1.85 mm of rail each side instead of 0.6.

Also decided: the status LED is three plain LEDs, not an addressable one. The
WS2812 family wants a supply above the only rail this board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
Parts:
- removed GND (x5): GND, symbol Custom:rail_down
- removed U2: TODO-BUCK-BOOST, symbol Device:U_TODO-BUCK-BOOST
- added GND (x4): GND, symbol Custom:rail_down
- added L2: 2.2µH, symbol Device:inductor_right
- added U2: TPS63001, symbol Device:U_TPS63001
Connections:
- net GND: now also C1.2, J2.2 (GND), U2.11 (EPAD), U2.3 (PGND), U2.7 (PSSYNC), U2.9 (GND)
- net V3V3: now also U2.1 (VOUT), U2.10 (FB); no longer U5.1 (VDD), U6.1 (VDD)
- net VBAT: now also U2.5 (VIN), U2.6 (EN), U2.8 (VINA)
- new net: L2.2, U2.2 (L2)
- new net: U5.1 (VDD), U6.1 (VDD)
- new net U2_L1: L2.1, U2.4 (L1)
